File: PCB/ppm.sch (KiCad schematic (older format))
At the start: 22 parts, among them U1 bq2403x

Commit message: Cleaning up code a bit
Other:
- note added: "R_SET = 1070 \Ohm [def charging current, R_SET = 2.5V * 450 / I_CHARG\nR_TMR = 60k \Ohm [time after which charging terminates for safety, ]\nR_DPPM = 37.7k \Ohm []\n\nThese can be not populated, or:\nR_CE = 0Ohm, Chip Enabled if USB present\nR_PSEL = 0Ohm, USB is primary source\nR_ISET2 = charge current for battery from USB, populate this one with 0Ohm to set 100mA\nR_ISET2H = or this one to set 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"
- note removed: "R_SET = 1070 \Ohm\nR_TMR = 60k \Ohm\nR_DPPM = 37.7k \Ohm\n\nThese can be not populated, or:\nR_CE = 10kOhm, Chip Enabled if USB present\nR_PSEL = 10kOhm, USB is primary source\nR_ISET2 = charge current for battery from USB, populate this one with 10kOhm to set 100mA\nR_ISET2H = or this one to set 500mA"
Changed lines of the file:
@@
 	6550 4600 6550 4550
 Text Notes 2700 2700 0    60   ~ 0
-R_SET = 1070 \Ohm\nR_TMR = 60k \Ohm\nR_DPPM = 37.7k \Ohm\n\nThese can be not populated, or:\nR_CE = 10kOhm, Chip Enabled if USB present\nR_PSEL  = 10kOhm, USB is primary source\nR_ISET2 = charge current for battery from USB, populate this one with 10kOhm to set 100mA\nR_ISET2H = or this one to set 500mA
+R_SET = 1070 \Ohm [def charging current, R_SET = 2.5V * 450 / I_CHARG\nR_TMR = 60k \Ohm [time after which charging terminates for safety, ]\nR_DPPM = 37.7k \Ohm []\n\nThese can be not populated, or:\nR_CE = 0Ohm, Chip Enabled if USB present\nR_PSEL  = 0Ohm, USB is primary source\nR_ISET2 = charge current for battery from USB, populate this one with 0Ohm to set 100mA\nR_ISET2H = or this one to set 500mA
 $Comp
 L C_Small C2
